File: hpboard/hpboard.kicad_sch (KiCad schematic)
At the start: 28 parts, among them Q1 T2N7002AK, Q2 T2N7002AK, Q3 Si4435FDY, Q4 Si4435FDY, SW1 FSM2JAH, U1 TMCS1108A4B, U2 ATtiny1604-SS, U3 TLV1117-50

Commit message: Less noise in current sensing. Faster regulation.
Parts:
- added C4: 100uF, Capacitor_Tantalum_SMD:CP_EIA-3528-21_Kemet-B_Pad1.50x2.35mm_HandSolder, symbol Device:C_Polarized_Small
- added C5, C6: 100nF, Capacitor_SMD:C_0603_1608Metric_Pad1.08x0.95mm_HandSolder, symbol Device:C_Small
- added R7, R8: 10k, Resistor_SMD:R_0805_2012Metric_Pad1.20x1.40mm_HandSolder, symbol Device:R_Small
- added R9: 1k, Resistor_SMD:R_0805_2012Metric_Pad1.20x1.40mm_HandSolder, symbol Device:R_Small
- C1: value 1uF -> 10uF
- C3: footprint Capacitor_SMD:C_0805_2012Metric_Pad1.18x1.45mm_HandSolder -> Capacitor_SMD:C_0603_1608Metric_Pad1.08x0.95mm_HandSolder
Connections:
- net +5V: now also C4.1, C5.2, R7.2, R8.2
- net GND: now also C4.2, C5.1, C6.2
- net SCL: now also R7.1
- net SDA: now also R8.1
- net SENSE_CURRENT: now also C6.1, R9.2; no longer U1.7 (VIOUT)
- new net: R9.1, U1.7 (VIOUT)

Commit message: Remove unnecessary pull-ups
Parts:
- removed R7, R8: 10k, Resistor_SMD:R_0805_2012Metric_Pad1.20x1.40mm_HandSolder, symbol Device:R_Small
Changed lines of the file:
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@@
   (junction (at 138.43 38.1) (diameter 0) (color 0 0 0 0)
   )
-  (junction (at 228.6 100.33) (diameter 0) (color 0 0 0 0)
-  )
   (junction (at 62.23 111.76) (diameter 0) (color 0 0 0 0)
   )
@@
   )
   (junction (at 115.57 48.26) (diameter 0) (color 0 0 0 0)
-  )
-  (junction (at 226.06 97.79) (diameter 0) (color 0 0 0 0)
   )
   (junction (at 114.3 129.54) (diameter 0) (color 0 0 0 0)
@@
     (stroke (width 0) (type default) (color 0 0 0 0))
   )
-  (wire (pts (xy 237.49 86.36) (xy 237.49 88.9))
-    (stroke (width 0) (type default) (color 0 0 0 0))
-  )
   (wire (pts (xy 157.48 148.59) (xy 157.48 110.49))
     (stroke (width 0) (type default) (color 0 0 0 0))
@@
     (stroke (width 0) (type default) (color 0 0 0 0))
   )
-  (wire (pts (xy 226.06 97.79) (xy 237.49 97.79))
-    (stroke (width 0) (type default) (color 0 0 0 0))
-  )
   (wire (pts (xy 224.79 161.29) (xy 165.1 161.29))
     (stroke (width 0) (type default) (color 0 0 0 0))
@@
     (stroke (width 0) (type default) (color 0 0 0 0))
   )
-  (wire (pts (xy 228.6 100.33) (xy 245.11 100.33))
-    (stroke (width 0) (type default) (color 0 0 0 0))
-  )
   (wire (pts (xy 41.91 158.75) (xy 54.61 158.75))
     (stroke (width 0) (type default) (color 0 0 0 0))
@@
     (stroke (width 0) (type default) (color 0 0 0 0))
   )
-  (wire (pts (xy 245.11 100.33) (xy 245.11 93.98))
-    (stroke (width 0) (type default) (color 0 0 0 0))
-  )
   (wire (pts (xy 54.61 158.75) (xy 54.61 166.37))
     (stroke (width 0) (type default) (color 0 0 0 0))
@@
     (stroke (width 0) (type default) (color 0 0 0 0))
   )
-  (wire (pts (xy 237.49 93.98) (xy 237.49 97.79))
-    (stroke (width 0) (type default) (color 0 0 0 0))
-  )
   (wire (pts (xy 38.1 38.1) (xy 53.34 38.1))
     (stroke (width 0) (type default) (color 0 0 0 0))
@@
   )
   (wire (pts (xy 114.3 129.54) (xy 114.3 132.08))
-    (stroke (width 0) (type default) (color 0 0 0 0))
-  )
-  (wire (pts (xy 245.11 86.36) (xy 245.11 88.9))
     (stroke (width 0) (type default) (color 0 0 0 0))
   )
@@
     (pin "2")
   )
-  (symbol (lib_id "power:+5V") (at 245.11 86.36 0) (unit 1)
-    (in_bom yes) (on_board yes)
-    (property "Reference" "#PWR02" (id 0) (at 245.11 90.17 0)
-      (effects (font (size 1.27 1.27)) hide)
-    )
-    (property "Value" "+5V" (id 1) (at 245.11 81.28 90))
-    (property "Footprint" "" (id 2) (at 245.11 86.36 0)
-      (effects (font (size 1.27 1.27)) hide)
-    )
-    (property "Datasheet" "" (id 3) (at 245.11 86.36 0)
-      (effects (font (size 1.27 1.27)) hide)
-    )
-    (pin "1")
-  )
   (symbol (lib_id "Regulator_Linear:TLV1117-50") (at 115.57 38.1 0) (unit 1)
     (in_bom yes) (on_board yes) (fields_autoplaced)
@@
     )
     (property "Datasheet" "~" (id 3) (at 85.09 52.07 0)
-      (effects (font (size 1.27 1.27)) hide)
-    )
-    (pin "1")
-    (pin "2")
-  )
-  (symbol (lib_id "power:+5V") (at 237.49 86.36 0) (unit 1)
-    (in_bom yes) (on_board yes)
-    (property "Reference" "#PWR01" (id 0) (at 237.49 90.17 0)
-      (effects (font (size 1.27 1.27)) hide)
-    )
-    (property "Value" "+5V" (id 1) (at 237.49 81.28 90))
-    (property "Footprint" "" (id 2) (at 237.49 86.36 0)
-      (effects (font (size 1.27 1.27)) hide)
-    )
-    (property "Datasheet" "" (id 3) (at 237.49 86.36 0)
-      (effects (font (size 1.27 1.27)) hide)
-    )
-    (pin "1")
-  )
-  (symbol (lib_id "Device:R_Small") (at 237.49 91.44 180) (unit 1)
-    (in_bom yes) (on_board yes) (fields_autoplaced)
-    (property "Reference" "R7" (id 0) (at 240.03 90.1699 0)
-      (effects (font (size 1.27 1.27)) (justify right))
-    )
-    (property "Value" "10k" (id 1) (at 240.03 92.7099 0)
-      (effects (font (size 1.27 1.27)) (justify right))
-    )
-    (property "Footprint" "Resistor_SMD:R_0805_2012Metric_Pad1.20x1.40mm_HandSolder" (id 2) (at 237.49 91.44 0)
-      (effects (font (size 1.27 1.27)) hide)
-    )
-    (property "Datasheet" "~" (id 3) (at 237.49 91.44 0)
       (effects (font (size 1.27 1.27)) hide)
     )
@@
     (pin "9")
   )
-  (symbol (lib_id "Device:R_Small") (at 245.11 91.44 180) (unit 1)
-    (in_bom yes) (on_board yes) (fields_autoplaced)
-    (property "Reference" "R8" (id 0) (at 247.65 90.1699 0)
-      (effects (font (size 1.27 1.27)) (justify right))
-    )
-    (property "Value" "10k" (id 1) (at 247.65 92.7099 0)
-      (effects (font (size 1.27 1.27)) (justify right))
-    )
-    (property "Footprint" "Resistor_SMD:R_0805_2012Metric_Pad1.20x1.40mm_HandSolder" (id 2) (at 245.11 91.44 0)
-      (effects (font (size 1.27 1.27)) hide)
-    )
-    (property "Datasheet" "~" (id 3) (at 245.11 91.44 0)
-      (effects (font (size 1.27 1.27)) hide)
-    )
-    (pin "1")
-    (pin "2")
-  )
   (symbol (lib_id "power:GND") (at 115.57 190.5 0) (unit 1)
     (in_bom yes) (on_board yes) (fields_autoplaced)
@@
       (reference "#FLG0102") (unit 1) (value "PWR_FLAG") (footprint "")
     )
-    (path "/77b0ab26-e022-43ff-b5b8-6194419d7931"
-      (reference "#PWR01") (unit 1) (value "+5V") (footprint "")
-    )
-    (path "/637f9519-cad1-477e-9485-c9772a96081e"
-      (reference "#PWR02") (unit 1) (value "+5V") (footprint "")
-    )
     (path "/00a722b4-7c0c-4cb1-9dbe-00bbf8eceb94"
       (reference "#PWR0101") (unit 1) (value "GND") (footprint "")
@@
       (reference "R6") (unit 1) (value "1k") (footprint "Resistor_SMD:R_0805_2012Metric_Pad1.20x1.40mm_HandSolder")
     )
-    (path "/80bd03bc-5fd8-4dd5-88b0-d25d065c2fb3"
-      (reference "R7") (unit 1) (value "10k") (footprint "Resistor_SMD:R_0805_2012Metric_Pad1.20x1.40mm_HandSolder")
-    )
-    (path "/d63e6680-0b44-494a-9400-47baf74304a3"
-      (reference "R8") (unit 1) (value "10k") (footprint "Resistor_SMD:R_0805_2012Metric_Pad1.20x1.40mm_HandSolder")
-    )
     (path "/711f03e7-e219-410a-aa64-06a260776d41"

Commit message: Rework PCB for better soldering
Parts:
- removed JPWR1: PJ-037BH, Library:PJ_037BH, symbol Connector:Barrel_Jack
- added JPWR1: Barrel_Jack_Switch, Connector_BarrelJack:BarrelJack_Horizontal, symbol Connector:Barrel_Jack_Switch
Connections:
- net 12V: now also JPWR1.1
- net GND: now also JPWR1.2, JPWR1.3
Changed lines of the file:
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@@
   (junction (at 127 48.26) (diameter 0) (color 0 0 0 0)
+  )
+  (junction (at 34.29 43.18) (diameter 0) (color 0 0 0 0)
   )
   (junction (at 38.1 38.1) (diameter 0) (color 0 0 0 0)
@@
     (stroke (width 0) (type default) (color 0 0 0 0))
   )
+  (wire (pts (xy 34.29 40.64) (xy 34.29 43.18))
+    (stroke (width 0) (type default) (color 0 0 0 0))
+  )
   (wire (pts (xy 123.19 38.1) (xy 127 38.1))
     (stroke (width 0) (type default) (color 0 0 0 0))
@@
     (stroke (width 0) (type default) (color 0 0 0 0))
   )
+  (wire (pts (xy 33.02 40.64) (xy 34.29 40.64))
+    (stroke (width 0) (type default) (color 0 0 0 0))
+  )
   (wire (pts (xy 53.34 71.12) (xy 55.88 71.12))
     (stroke (width 0) (type default) (color 0 0 0 0))
   )
-  (wire (pts (xy 38.1 43.18) (xy 33.02 43.18))
+  (wire (pts (xy 38.1 43.18) (xy 34.29 43.18))
     (stroke (width 0) (type default) (color 0 0 0 0))
   )
@@
   )
   (wire (pts (xy 115.57 48.26) (xy 127 48.26))
+    (stroke (width 0) (type default) (color 0 0 0 0))
+  )
+  (wire (pts (xy 34.29 43.18) (xy 33.02 43.18))
     (stroke (width 0) (type default) (color 0 0 0 0))
   )
@@
     )
     (property "Datasheet" "~" (id 3) (at 149.86 43.18 0)
-      (effects (font (size 1.27 1.27)) hide)
-    )
-    (pin "1")
-    (pin "2")
-  )
-  (symbol (lib_id "Connector:Barrel_Jack") (at 25.4 40.64 0) (unit 1)
-    (in_bom yes) (on_board yes) (fields_autoplaced)
-    (property "Reference" "JPWR1" (id 0) (at 25.4 31.75 0))
-    (property "Value" "PJ-037BH" (id 1) (at 25.4 34.29 0))
-    (property "Footprint" "Library:PJ_037BH" (id 2) (at 26.67 41.656 0)
-      (effects (font (size 1.27 1.27)) hide)
-    )
-    (property "Datasheet" "~" (id 3) (at 26.67 41.656 0)
       (effects (font (size 1.27 1.27)) hide)
     )
@@
     (pin "1")
     (pin "2")
+  )
+  (symbol (lib_id "Connector:Barrel_Jack_Switch") (at 25.4 40.64 0) (unit 1)
+    (in_bom yes) (on_board yes) (fields_autoplaced)
+    (property "Reference" "JPWR1" (id 0) (at 25.4 31.75 0))
+    (property "Value" "Barrel_Jack_Switch" (id 1) (at 25.4 34.29 0))
+    (property "Footprint" "Connector_BarrelJack:BarrelJack_Horizontal" (id 2) (at 26.67 41.656 0)
+      (effects (font (size 1.27 1.27)) hide)
+    )
+    (property "Datasheet" "~" (id 3) (at 26.67 41.656 0)
+      (effects (font (size 1.27 1.27)) hide)
+    )
+    (pin "1")
+    (pin "2")
+    (pin "3")
   )
   (symbol (lib_id "power:GND") (at 223.52 83.82 0) (unit 1)
@@
       (reference "JGND1") (unit 1) (value "Conn_01x01") (footprint "Library:MountingHole_3.2mm_Large")
     )
-    (path "/0cc169b4-c544-49dd-9342-96d29cadc80e"
-      (reference "JPWR1") (unit 1) (value "PJ-037BH") (footprint "Library:PJ_037BH")
+    (path "/97cd461e-91a1-41cc-923b-06b72ca1c308"
+      (reference "JPWR1") (unit 1) (value "Barrel_Jack_Switch") (footprint "Connector_BarrelJack:BarrelJack_Horizontal")
     )
     (path "/21c04f73-e593-4d54-88c0-de792dafa293"

Commit message: Add hole to PCB to allow the hotplate to SMD-solder its own clone. Switch GND and VCC on display module to support slimmer and more common variant
Connections:
- net +5V: now also JDISPLAY1.2 (Pin_2); no longer JDISPLAY1.1 (Pin_1)
- net GND: now also JDISPLAY1.1 (Pin_1); no longer JDISPLAY1.2 (Pin_2)
Changed lines of the file:
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@@
   (title_block
     (title "Heatplate controler")
-    (rev "1")
+    (rev "3")
   )
   (junction (at 138.43 38.1) (diameter 0) (color 0 0 0 0)
@@
     (pin "2")
   )
-  (symbol (lib_id "power:+5V") (at 220.98 82.55 180) (unit 1)
+  (symbol (lib_id "power:+5V") (at 223.52 83.82 180) (unit 1)
     (in_bom yes) (on_board yes)
-    (property "Reference" "#PWR0105" (id 0) (at 220.98 78.74 0)
-      (effects (font (size 1.27 1.27)) hide)
-    )
-    (property "Value" "+5V" (id 1) (at 220.98 87.63 90))
-    (property "Footprint" "" (id 2) (at 220.98 82.55 0)
-      (effects (font (size 1.27 1.27)) hide)
-    )
-    (property "Datasheet" "" (id 3) (at 220.98 82.55 0)
+    (property "Reference" "#PWR0105" (id 0) (at 223.52 80.01 0)
+      (effects (font (size 1.27 1.27)) hide)
+    )
+    (property "Value" "+5V" (id 1) (at 223.52 88.9 90))
+    (property "Footprint" "" (id 2) (at 223.52 83.82 0)
+      (effects (font (size 1.27 1.27)) hide)
+    )
+    (property "Datasheet" "" (id 3) (at 223.52 83.82 0)
       (effects (font (size 1.27 1.27)) hide)
     )
@@
     (pin "3")
   )
-  (symbol (lib_id "power:GND") (at 223.52 83.82 0) (unit 1)
+  (symbol (lib_id "power:GND") (at 220.98 82.55 0) (unit 1)
     (in_bom yes) (on_board yes)
-    (property "Reference" "#PWR0106" (id 0) (at 223.52 90.17 0)
-      (effects (font (size 1.27 1.27)) hide)
-    )
-    (property "Value" "GND" (id 1) (at 223.52 88.9 90))
-    (property "Footprint" "" (id 2) (at 223.52 83.82 0)
-      (effects (font (size 1.27 1.27)) hide)
-    )
-    (property "Datasheet" "" (id 3) (at 223.52 83.82 0)
-      (effects (font (size 1.27 1.27)) hide)
-    )
+    (property "Reference" "#PWR0106" (id 0) (at 220.98 88.9 0)
+      (effects (font (size 1.27 1.27)) hide)
+    )
+    (property "Value" "GND" (id 1) (at 220.98 87.63 90))
+    (property "Footprint" "" (id 2) (at 220.98 82.55 0)
+      (effects (font (size 1.27 1.27)) hide)
+    )
+    (property "Datasheet" "" (id 3) (at 220.98 82.55 0)
+      (effects (font (size 1.27 1.27)) hide)
+    )
